File: C.L.A.S/C.L.A.S.kicad_pcb (KiCad board)
At the start: 2 copper layers, 334.5 x 135.5 mm, 11 parts, among them J1 Screw_Terminal_01x02, J3 Conn_01x03_Pin, J4 Conn_01x03_Pin, J5 Conn_01x03_Pin, U1 ESP32-S3-DEVKITC-1-N8R2

Commit message: pcb_enclosure
Parts:
- added H1: MountingHole, MountingHole:MountingHole_3.2mm_M3, F.Cu at (82.0, 71.5)
- added H2: MountingHole, MountingHole:MountingHole_3.2mm_M3, F.Cu at (82.0, 186.6)
- added H3: MountingHole, MountingHole:MountingHole_3.2mm_M3, F.Cu at (393.0, 71.5)
- added H4: MountingHole, MountingHole:MountingHole_3.2mm_M3, F.Cu at (393.0, 186.6)
- added J2: Conn_01x03_Pin, Connector_PinHeader_2.54mm:PinHeader_1x03_P2.54mm_Vertical, F.Cu at (180.9, 73.0)
- moved J4 23.6 mm to (130.6, 73.0)
- moved J5 23.6 mm to (155.5, 73.0)
- moved J3 23.6 mm to (108.1, 73.5)
- moved Waterpump1 9.01 mm to (109.5, 178.5)
- moved peltier2 4.50 mm to (164.0, 178.0)
Connections:
- U1 pad J1_11: unconnected-(U1-GPIO18-PadJ1_11) -> Water_level
Routing:
- net Water_level: track 0.00 -> 79.4 mm, vias 0 -> 1
- net VCC_3v: track 212.8 -> 164.1 mm
- net Dht22: track 124.3 -> 99.2 mm
- net Soil: track 175.4 -> 151.6 mm
- net Waterpump: track 115.8 -> 107.1 mm
- net LDR: track 123.8 -> 116.0 mm
- net Peltier2: track 86.2 -> 84.3 mm
Other:
- board text added: "Water_level"

Commit message: BOM
Parts:
- added Waterpump2: ~, mosfet:MOSFET_KIT, F.Cu at (290.5, 157.0)
Connections:
- U1 pad J3_13: unconnected-(U1-GPIO35-PadJ3_13) -> grow
Routing:
- net grow: track 0.00 -> 75.9 mm, vias 0 -> 1
Other:
- board text added: "GrowLight"
Changed lines of the file:
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@@
 	(net 23 "Water_level")
 	(net 24 "unconnected-(U1-GPIO21-PadJ3_18)")
-	(net 25 "unconnected-(U1-GPIO35-PadJ3_13)")
+	(net 25 "grow")
 	(net 26 "unconnected-(U1-U0TXD{slash}GPIO43-PadJ3_2)")
 	(net 27 "unconnected-(U1-GPIO38-PadJ3_10)")
@@
 			(layers "*.Cu" "*.Mask")
 			(remove_unused_layers no)
-			(net 25 "unconnected-(U1-GPIO35-PadJ3_13)")
+			(net 25 "grow")
 			(pinfunction "GPIO35")
 			(pintype "bidirectional")
@@
 	(footprint "mosfet:MOSFET_KIT"
 		(layer "F.Cu")
+		(at 290.5 157)
+		(property "Reference" "Waterpump2"
+			(at -0.05 -11.75 0)
+			(unlocked yes)
+			(layer "F.SilkS")
+			(hide yes)
+			(effects
+				(font
+					(size 1 1)
+					(thickness 0.1)
+				)
+			)
+		)
+		(property "Value" "~"
+			(at -0.05 -10.2 0)
+			(unlocked yes)
+			(layer "F.Fab")
+			(effects
+				(font
+					(size 1 1)
+					(thickness 0.15)
+				)
+			)
+		)
+		(property "Datasheet" ""
+			(at 0 0 0)
+			(unlocked yes)
+			(layer "F.Fab")
+			(hide yes)
+			(effects
+				(font
+					(size 1 1)
+					(thickness 0.15)
+				)
+			)
+		)
+		(property "Description" ""
+			(at 0 0 0)
+			(unlocked yes)
+			(layer "F.Fab")
+			(hide yes)
+			(effects
+				(font
+					(size 1 1)
+					(thickness 0.15)
+				)
+			)
+		)
+		(sheetname "/")
+		(sheetfile "C.L.A.S.kicad_sch")
+		(attr smd)
+		(fp_rect
+			(start -17 -8.5)
+			(end 16.5 8.5)
+			(stroke
+				(width 0.1)
+				(type default)
+			)
+			(fill no)
+			(layer "F.SilkS")
+		)
+		(fp_rect
+			(start -15.5 -8.5)
+			(end -5.5 -1.5)
+			(stroke
+				(width 0.1)
+				(type default)
+			)
+			(fill no)
+			(layer "F.SilkS")
+		)
+		(fp_rect
+			(start -15.5 1.25)
+			(end -5.5 8.5)
+			(stroke
+				(width 0.1)
+				(type default)
+			)
+			(fill no)
+			(layer "F.SilkS")
+		)
+		(fp_rect
+			(start 12 -4.5)
+			(end 16.5 4.5)
+			(stroke
+				(width 0.1)
+				(type default)
+			)
+			(fill no)
+			(layer "F.SilkS")
+		)
+		(fp_text user "OUT"
+			(at -13.45 -3.4 0)
+			(unlocked yes)
+			(layer "F.SilkS")
+			(effects
+				(font
+					(size 2 2)
+					(thickness 0.1)
+				)
+				(justify left bottom)
+			)
+		)
+		(fp_text user "IN"
+			(at -9 3.5 180)
+			(unlocked yes)
+			(layer "F.SilkS")
+			(effects
+				(font
+					(size 2 2)
+					(thickness 0.1)
+				)
+				(justify left bottom)
+			)
+		)
+		(pad "1" thru_hole circle
+			(at 15 2.5)
+			(size 1.53 1.53)
+			(drill 1.02)
+			(layers "*.Cu" "*.Mask")
+			(remove_unused_layers no)
+			(net 2 "GND")
+			(pinfunction "GND")
+			(pintype "input")
+			(solder_mask_margin 0.102)
+		)
+		(pad "2" thru_hole circle
+			(at 15 -2.5 270)
+			(size 1.53 1.53)
+			(drill 1.02)
+			(layers "*.Cu" "*.Mask")
+			(remove_unused_layers no)
+			(net 25 "grow")
+			(pinfunction "PMW")
+			(pintype "input")
+			(solder_mask_margin 0.102)
+		)
+		(embedded_fonts no)
+		(model "D:/C.L.A.S/Libraries/PWM Mosfet Modul 400W.step"
+			(offset
+				(xyz 0 0 0)
+			)
+			(scale
+				(xyz 1 1 1)
+			)
+			(rotate
+				(xyz 0 0 0)
+			)
+		)
+	)
+	(footprint "mosfet:MOSFET_KIT"
+		(layer "F.Cu")
 		(at 127.5 132)
 		(property "Reference" "Peltier1"
@@
 	)
 	(gr_text "@YoussefAyman"
-		(at 268.5 175 0)
+		(at 236.5 183.5 0)
 		(layer "F.SilkS")
 		(effects
@@
 		)
 	)
+	(gr_text "GrowLight"
+		(at 289.5 170 0)
+		(layer "F.SilkS")
+		(effects
+			(font
+				(size 3 3)
+				(thickness 0.3)
+				(bold yes)
+				(italic yes)
+			)
+			(justify bottom)
+		)
+	)
 	(gr_text "Fan"
 		(at 378 77 0)
@@
 	)
 	(segment
+		(start 248.5 134.04)
+		(end 241.5 127.04)
+		(width 0.2)
+		(layer "F.Cu")
+		(net 25)
+	)
+	(segment
+		(start 248.5 135)
+		(end 248.5 134.04)
+		(width 0.2)
+		(layer "F.Cu")
+		(net 25)
+	)
+	(via
+		(at 248.5 135)
+		(size 0.6)
+		(drill 0.3)
+		(layers "F.Cu" "B.Cu")
+		(net 25)
+	)
+	(segment
+		(start 268 154.5)
+		(end 248.5 135)
+		(width 0.2)
+		(layer "B.Cu")
+		(net 25)
+	)
+	(segment
+		(start 305.5 154.5)
+		(end 268 154.5)
+		(width 0.2)
+		(layer "B.Cu")
+		(net 25)
+	)
+	(segment
