File: C.L.A.S/C.L.A.S.kicad_sch (KiCad schematic)
At the start: 27 parts, among them J1 Screw_Terminal_01x02, J3 Conn_01x03_Pin, J4 Conn_01x03_Pin, J5 Conn_01x03_Pin, M1 Fan, M2 Motor_DC, M3 Fan, M4 Fan, M5 Fan, M6 Fan, U1 ESP32-S3-DEVKITC-1-N8R2, U2 DHT22

Commit message: PCB
Parts:
- Fan1, Heatlamp1, Humidifer1, Peltier1, Waterpump1, peltier2: footprint Library:MOSFET_KIT -> mosfet:MOSFET_KIT
- J1: footprint (none) -> TerminalBlock_Phoenix:TerminalBlock_Phoenix_MKDS-1,5-2-5.08_1x02_P5.08mm_Horizontal
- U2: footprint Sensor:Aosong_DHT11_5.5x12.0_P2.54mm -> (none)
Changed lines of the file:
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@@
 			)
 		)
-		(property "Footprint" "Library:MOSFET_KIT"
+		(property "Footprint" "mosfet:MOSFET_KIT"
 			(at 318.77 250.19 0)
 			(effects
@@
 			)
 		)
-		(property "Footprint" "Library:MOSFET_KIT"
+		(property "Footprint" "mosfet:MOSFET_KIT"
 			(at 323.85 198.12 0)
 			(effects
@@
 			)
 		)
-		(property "Footprint" "Sensor:Aosong_DHT11_5.5x12.0_P2.54mm"
+		(property "Footprint" ""
 			(at 326.39 378.46 0)
 			(effects
@@
 			)
 		)
-		(property "Footprint" "Library:MOSFET_KIT"
+		(property "Footprint" "mosfet:MOSFET_KIT"
 			(at 234.95 247.65 0)
 			(effects
@@
 			)
 		)
-		(property "Footprint" "Library:MOSFET_KIT"
+		(property "Footprint" "mosfet:MOSFET_KIT"
 			(at 234.95 198.12 0)
 			(effects
@@
 			)
 		)
-		(property "Footprint" "Library:MOSFET_KIT"
+		(property "Footprint" "mosfet:MOSFET_KIT"
 			(at 151.13 245.11 0)
 			(effects
@@
 			)
 		)
-		(property "Footprint" "Library:MOSFET_KIT"
+		(property "Footprint" "mosfet:MOSFET_KIT"
 			(at 138.43 194.31 0)
 			(effects
@@
 			)
 		)
-		(property "Footprint" ""
+		(property "Footprint" "TerminalBlock_Phoenix:TerminalBlock_Phoenix_MKDS-1,5-2-5.08_1x02_P5.08mm_Horizontal"
 			(at 175.26 340.36 0)
 			(effects

Commit message: pcb_enclosure
Parts:
- added H1, H2, H3, H4: MountingHole, MountingHole:MountingHole_3.2mm_M3, symbol Mechanical:MountingHole
- added J2: Conn_01x03_Pin, Connector_PinHeader_2.54mm:PinHeader_1x03_P2.54mm_Vertical, symbol Connector:Conn_01x03_Pin
- added U3: ~, symbol New_Library:Water_Level
Connections:
- net GND: now also J2.3 (Pin_3), U3. (Signal)
- net VCC: now also J2.2 (Pin_2), U3. (Signal)
- net Water_level: now reaches U1.J1_11 (GPIO18)
- net Water_level: now also J2.1 (Pin_1), U3. (Signal)
Other:
- note added: "M3 mounting holes"
- note added: "Water_Level"
- note added: "Waterlevel"
- moved on the sheet: J4, J5, LDR1

Commit message: BOM
Parts:
- added Waterpump2: ~, mosfet:MOSFET_KIT, symbol New_Library:Mosfet_Controller
Connections:
- net GND: now also Waterpump2. (IN-), Waterpump2.1 (GND); no longer GrowLight1. (GND)
- net VCC: now also Waterpump2. (IN-); no longer GrowLight1. (GND)
- net grow: now also U1.J3_13 (GPIO35), Waterpump2.2 (PMW)
- new net GND_grow: GrowLight1. (GND), Waterpump2. (IN-)
- new net VCC_grow: GrowLight1. (GND), Waterpump2. (IN-)
